Commit message: add rgbd + 3dlidar.

File: rofa/ros2_ws/src/my_robot_description/urdf/robot.urdf.xacro (robot description, xacro)
@@ -121,18 +121,109 @@
     <origin xyz="-0.15 0 0.02" rpy="0 0 0"/>
   </joint>
-  <!-- future camera mount -->
+  <!-- RGBD camera mount -->
   <link name="camera_mount_link"/>
   <joint name="camera_mount_joint" type="fixed">
     <parent link="base_link"/>
     <child link="camera_mount_link"/>
-    <origin xyz="0.15 0.0 0.20" rpy="0 0 0"/>
-  </joint>
-  <!-- future lidar mount -->
-  <link name="lidar_link"/>
-  <joint name="lidar_joint" type="fixed">
-    <parent link="base_link"/>
-    <child link="lidar_link"/>
+    <origin xyz="0.0 0.0 0.60" rpy="0 0 0"/>
+  </joint>
+  <!-- camera body -->
+  <link name="camera_link">
+    <inertial>
+      <origin xyz="0 0 0" rpy="0 0 0"/>
+      <mass value="0.2"/>
+      <inertia ixx="0.0001" ixy="0.0" ixz="0.0"
+               iyy="0.0001" iyz="0.0"
+               izz="0.0001"/>
+    </inertial>
+    <visual>
+      <origin xyz="0 0 0" rpy="0 0 0"/>
+      <geometry>
+        <box size="0.09 0.025 0.025"/>
+      </geometry>
+      <material name="dark_gray">
+        <color rgba="0.25 0.25 0.25 1.0"/>
+      </material>
+    </visual>
+    <collision>
+      <origin xyz="0 0 0" rpy="0 0 0"/>
+      <geometry>
+        <box size="0.09 0.025 0.025"/>
+      </geometry>
+    </collision>
+  </link>
+  <gazebo reference="camera_link">
+    <material>Gazebo/DarkGrey</material>
+  </gazebo>
+  <joint name="camera_joint" type="fixed">
+    <parent link="camera_mount_link"/>
+    <child link="camera_link"/>
+    <origin xyz="0 0 0" rpy="0 0 0"/>
+  </joint>
+  <!-- color frame -->
+  <link name="camera_color_frame"/>
+  <joint name="camera_color_joint" type="fixed">
+    <parent link="camera_link"/>
+    <child link="camera_color_frame"/>
+    <origin xyz="0 0 0" rpy="0 0 0"/>
+  </joint>
+  <link name="camera_color_optical_frame"/>
+  <joint name="camera_color_optical_joint" type="fixed">
+    <parent link="camera_color_frame"/>
+    <child link="camera_color_optical_frame"/>
+    <origin xyz="0 0 0" rpy="-1.57079632679 0 -1.57079632679"/>
+  </joint>
+  <!-- depth frame -->
+  <link name="camera_depth_frame"/>
+  <joint name="camera_depth_joint" type="fixed">
+    <parent link="camera_link"/>
+    <child link="camera_depth_frame"/>
+    <origin xyz="0 0 0" rpy="0 0 0"/>
+  </joint>
+  <link name="camera_depth_optical_frame"/>
+  <joint name="camera_depth_optical_joint" type="fixed">
+    <parent link="camera_depth_frame"/>
+    <child link="camera_depth_optical_frame"/>
+    <origin xyz="0 0 0" rpy="-1.57079632679 0 -1.57079632679"/>
+  </joint>
+  <!-- MID-360 approximate mount -->
+  <link name="mid360_link">
+    <inertial>
+      <origin xyz="0 0 0" rpy="0 0 0"/>
+      <mass value="0.265"/>
+      <inertia ixx="0.0002" ixy="0.0" ixz="0.0"
+               iyy="0.0002" iyz="0.0"
+               izz="0.0002"/>
+    </inertial>
+    <visual>
+      <origin xyz="0 0 0" rpy="0 0 0"/>
+      <geometry>
+        <cylinder radius="0.0325" length="0.06"/>
+      </geometry>
+      <material name="mid360_gray">
+        <color rgba="0.35 0.35 0.35 1.0"/>
+      </material>
+    </visual>
+    <collision>
+      <origin xyz="0 0 0" rpy="0 0 0"/>
+      <geometry>
+        <cylinder radius="0.0325" length="0.06"/>
+      </geometry>
+    </collision>
+  </link>
+  <joint name="mid360_joint" type="fixed">
+    <parent link="base_link"/>
+    <child link="mid360_link"/>
     <origin xyz="0.0 0.0 0.28" rpy="0 0 0"/>
   </joint>
+  <link name="mid360_frame"/>
+  <joint name="mid360_frame_joint" type="fixed">
+    <parent link="mid360_link"/>
+    <child link="mid360_frame"/>
+    <origin xyz="0 0 0" rpy="0 0 0"/>
+  </joint>
+  <gazebo reference="mid360_link">
+    <material>Gazebo/DarkGrey</material>
+  </gazebo>
   <!-- friction -->
   <gazebo reference="left_wheel_link">
@@ -166,3 +257,78 @@
     </plugin>
   </gazebo>
+  <!-- Gazebo RGBD camera -->
+  <gazebo reference="camera_link">
+    <sensor name="rgbd_camera" type="depth">
+      <always_on>true</always_on>
+      <update_rate>30.0</update_rate>
+      <visualize>false</visualize>
+      <camera>
+        <horizontal_fov>1.211259</horizontal_fov>
+        <image>
+          <width>640</width>
+          <height>480</height>
+          <format>R8G8B8</format>
+        </image>
+        <clip>
+          <near>0.1</near>
+          <far>8.0</far>
+        </clip>
+      </camera>
+      <plugin name="gazebo_ros_camera" filename="libgazebo_ros_camera.so">
+        <ros>
+          <namespace>/camera</namespace>
+          <remapping>image_raw:=color/image_raw</remapping>
+          <remapping>camera_info:=color/camera_info</remapping>
+          <remapping>depth/image_raw:=depth/image_rect_raw</remapping>
+          <remapping>depth/camera_info:=depth/camera_info</remapping>
+          <remapping>points:=depth/color/points</remapping>
+        </ros>
+        <frame_name>camera_color_optical_frame</frame_name>
+        <min_depth>0.1</min_depth>
+        <max_depth>8.0</max_depth>
+      </plugin>
+    </sensor>
+  </gazebo>
+  <!-- Gazebo MID-360 approximate lidar -->
+  <gazebo reference="mid360_link">
+    <sensor name="mid360_lidar" type="ray">
+      <always_on>true</always_on>
+      <update_rate>10.0</update_rate>
+      <visualize>false</visualize>
+      <ray>
+        <scan>
+          <horizontal>
+            <samples>1000</samples>
+            <resolution>1.0</resolution>
+            <min_angle>-3.14159265359</min_angle>
+            <max_angle>3.14159265359</max_angle>
+          </horizontal>
+          <vertical>
+            <samples>20</samples>
+            <resolution>1.0</resolution>
+            <min_angle>-0.122173</min_angle>
+            <max_angle>0.907571</max_angle>
+          </vertical>
+        </scan>
+        <range>
+          <min>0.1</min>
+          <max>40.0</max>
+          <resolution>0.01</resolution>
+        </range>
+        <noise>
+          <type>gaussian</type>
+          <mean>0.0</mean>
+          <stddev>0.01</stddev>
+        </noise>
+      </ray>
+      <plugin name="mid360_pointcloud" filename="libgazebo_ros_ray_sensor.so">
+        <ros>
+          <namespace>/livox</namespace>
+          <remapping>~/out:=points</remapping>
+        </ros>
+        <output_type>sensor_msgs/PointCloud2</output_type>
+        <frame_name>mid360_frame</frame_name>
+      </plugin>
+    </sensor>
+  </gazebo>
 </robot>

Commit message: basic RGBD + 3DLidar. tested.

File: rofa/ros2_ws/src/my_robot_description/urdf/robot.urdf.xacro (robot description, xacro)
@@ -140,5 +140,5 @@
       <origin xyz="0 0 0" rpy="0 0 0"/>
       <geometry>
-        <box size="0.09 0.025 0.025"/>
+        <box size="0.025 0.09 0.025"/>
       </geometry>
       <material name="dark_gray">
@@ -187,6 +187,6 @@
     <origin xyz="0 0 0" rpy="-1.57079632679 0 -1.57079632679"/>
   </joint>
-  <!-- MID-360 approximate mount -->
-  <link name="mid360_link">
+  <!-- 3D lidar mount -->
+  <link name="lidar_link">
     <inertial>
       <origin xyz="0 0 0" rpy="0 0 0"/>
@@ -201,5 +201,5 @@
         <cylinder radius="0.0325" length="0.06"/>
       </geometry>
-      <material name="mid360_gray">
+      <material name="lidar_gray">
         <color rgba="0.35 0.35 0.35 1.0"/>
       </material>
@@ -212,16 +212,16 @@
     </collision>
   </link>
-  <joint name="mid360_joint" type="fixed">
-    <parent link="base_link"/>
-    <child link="mid360_link"/>
+  <joint name="lidar_joint" type="fixed">
+    <parent link="base_link"/>
+    <child link="lidar_link"/>
     <origin xyz="0.0 0.0 0.28" rpy="0 0 0"/>
   </joint>
-  <link name="mid360_frame"/>
-  <joint name="mid360_frame_joint" type="fixed">
-    <parent link="mid360_link"/>
-    <child link="mid360_frame"/>
-    <origin xyz="0 0 0" rpy="0 0 0"/>
-  </joint>
-  <gazebo reference="mid360_link">
+  <link name="lidar_frame"/>
+  <joint name="lidar_frame_joint" type="fixed">
+    <parent link="lidar_link"/>
+    <child link="lidar_frame"/>
+    <origin xyz="0 0 0" rpy="0 0 0"/>
+  </joint>
+  <gazebo reference="lidar_link">
     <material>Gazebo/DarkGrey</material>
   </gazebo>
@@ -259,5 +259,5 @@
   <!-- Gazebo RGBD camera -->
   <gazebo reference="camera_link">
-    <sensor name="rgbd_camera" type="depth">
+    <sensor name="rgbd_sensor" type="depth">
       <always_on>true</always_on>
       <update_rate>30.0</update_rate>
@@ -277,12 +277,13 @@
       <plugin name="gazebo_ros_camera" filename="libgazebo_ros_camera.so">
         <ros>
-          <namespace>/camera</namespace>
-          <remapping>image_raw:=color/image_raw</remapping>
-          <remapping>camera_info:=color/camera_info</remapping>
-          <remapping>depth/image_raw:=depth/image_rect_raw</remapping>
-          <remapping>depth/camera_info:=depth/camera_info</remapping>
-          <remapping>points:=depth/color/points</remapping>
+          <namespace>/</namespace>
+          <remapping>rgbd/image_raw:=rgbd/image_raw</remapping>
+          <remapping>rgbd/camera_info:=rgbd/camera_info</remapping>
+          <remapping>rgbd/depth/image_raw:=rgbd/depth/image_raw</remapping>
+          <remapping>rgbd/depth/camera_info:=rgbd/depth/camera_info</remapping>
+          <remapping>rgbd/points:=rgbd/points</remapping>
         </ros>
-        <frame_name>camera_color_optical_frame</frame_name>
+        <camera_name>rgbd</camera_name>
+        <frame_name>camera_depth_optical_frame</frame_name>
         <min_depth>0.1</min_depth>
         <max_depth>8.0</max_depth>
@@ -290,7 +291,7 @@
     </sensor>
   </gazebo>
-  <!-- Gazebo MID-360 approximate lidar -->
-  <gazebo reference="mid360_link">
-    <sensor name="mid360_lidar" type="ray">
+  <!-- Gazebo 3D lidar -->
+  <gazebo reference="lidar_link">
+    <sensor name="lidar_sensor" type="ray">
       <always_on>true</always_on>
       <update_rate>10.0</update_rate>
@@ -322,11 +323,11 @@
         </noise>
       </ray>
-      <plugin name="mid360_pointcloud" filename="libgazebo_ros_ray_sensor.so">
+      <plugin name="lidar_pointcloud" filename="libgazebo_ros_ray_sensor.so">
         <ros>
-          <namespace>/livox</namespace>
+          <namespace>/lidar</namespace>
           <remapping>~/out:=points</remapping>
         </ros>
         <output_type>sensor_msgs/PointCloud2</output_type>
-        <frame_name>mid360_frame</frame_name>
+        <frame_name>lidar_frame</frame_name>
       </plugin>
     </sensor>
